File: src/sch/norsid.sch (EAGLE design)
At the start: 6 parts, among them Q1 16MHz, U1 ATMEGA2560-16AU

Commit message: Schematic fixed
Parts:
- added C3: 1u, capacitor-wima:C2.5/2
- added X1: LINE OUT, con-hirschmann:TOBU3
- renumbered U$1 to U2
Connections:
- new net CS: U1.(A13)PC5, U2.#CS
- new net N$3: U2.AUDIO_IN, U2.GND, U2.POTX, U2.POTY, X1.2
- new net N$4: U1.(OC1A/PCINT5)PB5, U2.CLOCK
- new net N$5: C3.1, U2.AUDIO_OUT
- new net N$6: C3.2, X1.1
- new net RES: U1.(A15)PC7, U2.RESET
- new net RW: U1.(A14)PC6, U2.R/W
- net A0: now also U1.(A8)PC0
- net A1: now also U1.(A9)PC1
- net A2: now also U1.(A10)PC2
- net A3: now also U1.(A11)PC3
- net A4: now also U1.(A12)PC4
- net D0: now also U1.(AD0)PA0
- net D1: now also U1.(AD1)PA1
- net D2: now also U1.(AD2)PA2
- net D3: now also U1.(AD3)PA3
- net D4: now also U1.(AD4)PA4
- net D5: now also U1.(AD5)PA5
- net D6: now also U1.(AD6)PA6
- net D7: now also U1.(AD7)PA7
- net GND: no longer U2.GND
Other:
- note added: "6581"
- note added: "U2"

Commit message: Updating schematic
Parts:
- added R1: 1K, ngspice-simulation:R
- renumbered C9 to C4
Connections:
- new net N$7: C3.2, R1.2
- net N$6: now also R1.1; no longer C3.2
Other:
- moved on the sheet: X1
Changed lines of the file:
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@@
 <part name="GND6" library="supply1" deviceset="GND" device=""/>
 <part name="P+10" library="supply1" deviceset="+5V" device=""/>
-<part name="C9" library="capacitor-wima" deviceset="C" device="2.5/2" value="100n"/>
+<part name="C4" library="capacitor-wima" deviceset="C" device="2.5/2" value="100n"/>
 <part name="Q1" library="crystal" library_urn="urn:adsk.eagle:library:204" deviceset="CRYSTAL" device="HC49U70" package3d_urn="urn:adsk.eagle:package:12079/1" value="16MHz"/>
 <part name="GND2" library="supply1" deviceset="GND" device=""/>
 <part name="C3" library="capacitor-wima" deviceset="C" device="2.5/2" value="1u"/>
 <part name="X1" library="con-hirschmann" library_urn="urn:adsk.eagle:library:153" deviceset="TOBU3" device="" package3d_urn="urn:adsk.eagle:package:7468/1" value="LINE OUT"/>
+<part name="R1" library="ngspice-simulation" library_urn="urn:adsk.eagle:library:527439" deviceset="R" device="" value="1K"/>
 </parts>
 <sheets>
@@
 <attribute name="VALUE" x="-93.98" y="144.78" size="1.778" layer="96" rot="R180"/>
 </instance>
-<instance part="C9" gate="G$1" x="-96.52" y="129.54" smashed="yes" rot="R180">
+<instance part="C4" gate="G$1" x="-96.52" y="129.54" smashed="yes" rot="R180">
 <attribute name="NAME" x="-98.044" y="129.159" size="1.778" layer="95" rot="R180"/>
 <attribute name="VALUE" x="-98.044" y="134.239" size="1.778" layer="96" rot="R180"/>
@@
 <attribute name="VALUE" x="-93.98" y="160.02" size="1.778" layer="96" rot="R180"/>
 </instance>
-<instance part="GND2" gate="1" x="73.66" y="109.22" smashed="yes">
-<attribute name="VALUE" x="81.28" y="111.76" size="1.778" layer="96" rot="R180"/>
+<instance part="GND2" gate="1" x="73.66" y="101.6" smashed="yes">
+<attribute name="VALUE" x="71.12" y="104.14" size="1.778" layer="96" rot="R180"/>
 </instance>
 <instance part="C3" gate="G$1" x="83.82" y="116.84" smashed="yes" rot="R90">
@@
 <attribute name="VALUE" x="85.979" y="120.904" size="1.778" layer="96" rot="R180"/>
 </instance>
-<instance part="X1" gate="B" x="91.44" y="116.84" smashed="yes" rot="MR0">
-<attribute name="NAME" x="92.964" y="118.11" size="1.778" layer="95" rot="MR0"/>
-<attribute name="VALUE" x="106.68" y="114.3" size="1.778" layer="96" rot="MR0"/>
+<instance part="X1" gate="B" x="93.98" y="106.68" smashed="yes" rot="MR0">
+<attribute name="NAME" x="100.584" y="107.95" size="1.778" layer="95" rot="MR0"/>
+<attribute name="VALUE" x="109.22" y="104.14" size="1.778" layer="96" rot="MR0"/>
+</instance>
+<instance part="R1" gate="G$1" x="88.9" y="111.76" smashed="yes" rot="R90">
+<attribute name="NAME" x="86.36" y="111.76" size="1.778" layer="95" rot="R180"/>
+<attribute name="VALUE" x="86.36" y="107.95" size="1.778" layer="96" rot="R180"/>
 </instance>
 </instances>
@@
 <wire x1="-86.36" y1="119.38" x2="-91.44" y2="119.38" width="0.1524" layer="91"/>
 <junction x="-91.44" y="119.38"/>
-<pinref part="C9" gate="G$1" pin="1"/>
+<pinref part="C4" gate="G$1" pin="1"/>
 <wire x1="-96.52" y1="127" x2="-91.44" y2="127" width="0.1524" layer="91"/>
 </segment>
@@
 <wire x1="-91.44" y1="132.08" x2="-91.44" y2="134.62" width="0.1524" layer="91"/>
 <junction x="-91.44" y="134.62"/>
-<pinref part="C9" gate="G$1" pin="2"/>
+<pinref part="C4" gate="G$1" pin="2"/>
 <wire x1="-96.52" y1="134.62" x2="-91.44" y2="134.62" width="0.1524" layer="91"/>
 </segment>
@@
 <pinref part="U2" gate="G$1" pin="POTY"/>
 <wire x1="73.66" y1="124.46" x2="73.66" y2="119.38" width="0.1524" layer="91"/>
-<wire x1="73.66" y1="119.38" x2="73.66" y2="114.3" width="0.1524" layer="91"/>
-<wire x1="73.66" y1="114.3" x2="73.66" y2="111.76" width="0.1524" layer="91"/>
+<wire x1="73.66" y1="119.38" x2="73.66" y2="104.14" width="0.1524" layer="91"/>
 <wire x1="60.96" y1="124.46" x2="73.66" y2="124.46" width="0.1524" layer="91"/>
 <junction x="73.66" y="124.46"/>
@@
 <junction x="73.66" y="127"/>
 <pinref part="X1" gate="B" pin="2"/>
-<wire x1="88.9" y1="114.3" x2="73.66" y2="114.3" width="0.1524" layer="91"/>
-<junction x="73.66" y="114.3"/>
+<wire x1="91.44" y1="104.14" x2="73.66" y2="104.14" width="0.1524" layer="91"/>
+<junction x="73.66" y="104.14"/>
 </segment>
 </net>
@@
 <net name="N$6" class="0">
 <segment>
+<pinref part="X1" gate="B" pin="1"/>
+<wire x1="88.9" y1="106.68" x2="91.44" y2="106.68" width="0.1524" layer="91"/>
+<pinref part="R1" gate="G$1" pin="1"/>
+</segment>
+</net>
+<net name="N$7" class="0">
+<segment>
 <pinref part="C3" gate="G$1" pin="2"/>
-<pinref part="X1" gate="B" pin="1"/>
+<pinref part="R1" gate="G$1" pin="2"/>
 </segment>
 </net>
@@
 packages will not be understood (or retained) with this version.
 </note>
+<note version="8.4" severity="warning">
+Since Version 8.4, EAGLE supports properties for SPICE simulation.
+Probes in schematics and SPICE mapping objects found in parts and library devices
+will not be understood with this version. Update EAGLE to the latest version
+for full support of SPICE simulation.
+</note>
 </compatibility>
